File: clasicOverdrive.kicad_pcb (KiCad board)
At the start: 2 copper layers, 41 x 77 mm, 58 parts, among them J1 Jack-DC, J2 AudioJack3_Switch, J3 AudioJack3_Switch, Q1 2N2222, Q2 2N2222, T1 LA_LOGO, U1 foot_switch, U2 LM4562

Commit message: Rev-A Fabricated 2019_12_01
Parts:
- added G***: LOGO, clasicOverdrive:clasicOverdrive_QR, F.Cu at (138.0, 132.8)
- moved R11 1.20 mm to (127.7, 97.4)
- moved TP2 0.16 mm to (129.0, 117.7)
Routing:
- net +4V5: track 56.7 -> 55.3 mm

Commit message: Rev A - fabrication 2: silkscreen QR and website
Parts:
- removed the G*** at (138.0, 132.8)
- added G***: LOGO, clasicOverdrive:clasicOverdrive_QR_silk, F.Cu at (138.0, 132.8)
Other:
- board text added: "github.com/ leardilap/ clasicOverdrive"
