File: clasicOverdrive.sch (KiCad schematic (older format))
At the start: 43 parts, among them J1 Jack-DC, J2 Audio-Jack-3, J3 Audio-Jack-2, Q1 2N2222, Q2 2N2222, U1 foot_switch, U2 LM4562

Commit message: annotate and footprint assignment init
Parts:
- C1: value C -> 22n; footprint (none) -> Capacitor_SMD:C_0805_2012Metric_Pad1.15x1.50mm_HandSolder
- C10: value C -> 0.1u; footprint (none) -> Capacitor_SMD:C_0805_2012Metric_Pad1.15x1.50mm_HandSolder
- C11: value CP -> 10u; footprint (none) -> Capacitor_SMD:C_1206_3216Metric_Pad1.24x1.80mm_HandSolder
- C2: value C -> 47 n; footprint (none) -> Capacitor_SMD:C_0805_2012Metric_Pad1.15x1.50mm_HandSolder
- C3, C9: value C -> 1u; footprint (none) -> Capacitor_SMD:C_0805_2012Metric_Pad1.15x1.50mm_HandSolder
- C4: value C -> 51p; footprint (none) -> Capacitor_SMD:C_0805_2012Metric_Pad1.15x1.50mm_HandSolder
- C5: value CP -> 100u; footprint (none) -> Capacitor_SMD:C_1206_3216Metric_Pad1.24x1.80mm_HandSolder
- C6, C7: value CP -> 0.22u; footprint (none) -> Capacitor_SMD:C_1206_3216Metric_Pad1.24x1.80mm_HandSolder
- C8: value CP -> 47u; footprint (none) -> Capacitor_SMD:C_1206_3216Metric_Pad1.24x1.80mm_HandSolder
- D1: footprint (none) -> LED_SMD:LED_1206_3216Metric_Pad1.07x1.80mm_HandSolder
- D2, D3: footprint Diode_THT:D_DO-35_SOD27_Horizontal_RM10 -> Diode_SMD:D_0805_2012Metric_Pad0.97x1.50mm_HandSolder
- R1, R6: value R -> 4.7k; footprint (none) -> Resistor_SMD:R_0603_1608Metric_Pad0.84x1.00mm_HandSolder
- R10, R11, R13, R17, R5, R7: value R -> 10k; footprint (none) -> Resistor_SMD:R_0603_1608Metric_Pad0.84x1.00mm_HandSolder
- R12: value R -> 220; footprint (none) -> Resistor_SMD:R_0603_1608Metric_Pad0.84x1.00mm_HandSolder
- R14, R15, R3, R9: value R -> 1k; footprint (none) -> Resistor_SMD:R_0603_1608Metric_Pad0.84x1.00mm_HandSolder
- R16, R2, R4: value R -> 511k; footprint (none) -> Resistor_SMD:R_0603_1608Metric_Pad0.84x1.00mm_HandSolder
- R18: value R -> 100; footprint (none) -> Resistor_SMD:R_0603_1608Metric_Pad0.84x1.00mm_HandSolder
- R19: footprint (none) -> Resistor_SMD:R_0603_1608Metric_Pad0.84x1.00mm_HandSolder
- R8: value R -> 51k; footprint (none) -> Resistor_SMD:R_0603_1608Metric_Pad0.84x1.00mm_HandSolder
- RV1: value POT -> 500k
- RV2: value POT -> 25k
- RV3: value POT -> 100k
Other:
- note added: "DRIVE"
- note added: "TONE"
- note added: "tant"

Commit message: all footprints added and layout of pcb complete
Parts:
- removed J2: Audio-Jack-3, symbol Connector_Specialized:Audio-Jack-3
- removed J3: Audio-Jack-2, symbol Connector_Specialized:Audio-Jack-2
- added CON1, CON2: SN49B12B, digikey-footprints:Headphone_Jack_6.35mm_RA49B14B, symbol dk_Barrel-Audio-Connectors:SN49B12B
- J1: footprint (none) -> Connector_Audio:Jack_Horizontal
- Q1, Q2: footprint Package_TO_SOT_THT:TO-18 -> Package_TO_SOT_THT:TO-18-3
- RV1, RV2, RV3: footprint (none) -> clasicOverdrive:Pot_series_296
- U1: footprint (none) -> clasicOverdrive:FS57003PLT2B2M2QE
Connections:
- wire segments 118 -> 119
Other:
- note added: "LEVEL"
Changed lines of the file:
@@
 F 0 "RV3" H 7480 2796 50  0000 R CNN
 F 1 "100k" H 7480 2705 50  0000 R CNN
-F 2 "" H 7550 2750 50  0001 C CNN
+F 2 "clasicOverdrive:Pot_series_296" H 7550 2750 50  0001 C CNN
 F 3 "~" H 7550 2750 50  0001 C CNN
 	1    7550 2750
@@
 F 0 "Q2" H 8591 2796 50  0000 L CNN
 F 1 "2N2222" H 8600 2700 50  0000 L CNN
-F 2 "Package_TO_SOT_THT:TO-18" H 8600 2675 50  0001 L CIN
+F 2 "Package_TO_SOT_THT:TO-18-3" H 8600 2675 50  0001 L CIN
 F 3 "https://www.centralsemi.com/get_document.php?cmp=1&mergetype=pd&mergepath=pd&pdf_id=2N2221.PDF" H 8400 2750 50  0001 L CNN
 	1    8400 2750
@@
 F 0 "RV2" V 5350 1650 50  0000 R CNN
 F 1 "25k" V 5450 1650 50  0000 R CNN
-F 2 "" H 5550 1600 50  0001 C CNN
+F 2 "clasicOverdrive:Pot_series_296" H 5550 1600 50  0001 C CNN
 F 3 "~" H 5550 1600 50  0001 C CNN
 	1    5550 1600
@@
 F 0 "RV1" V 4350 2600 50  0000 R CNN
 F 1 "500k" V 4450 2600 50  0000 R CNN
-F 2 "" H 4550 2550 50  0001 C CNN
+F 2 "clasicOverdrive:Pot_series_296" H 4550 2550 50  0001 C CNN
 F 3 "~" H 4550 2550 50  0001 C CNN
 	1    4550 2550
@@
 $EndComp
 $Comp
-L Connector_Specialized:Audio-Jack-2 J3
-U 1 1 5ACC4995
-P 10600 2900
-F 0 "J3" H 10607 3125 50  0000 C CNN
-F 1 "Audio-Jack-2" H 10607 3034 50  0000 C CNN
-F 2 "" H 10850 2900 50  0001 C CNN
-F 3 "~" H 10850 2900 50  0001 C CNN
-	1    10600 2900
-	-1   0    0    -1
-$EndComp
-$Comp
-L Connector_Specialized:Audio-Jack-3 J2
-U 1 1 5ACC4D69
-P 900 3700
-F 0 "J2" H 876 4025 50  0000 C CNN
-F 1 "Audio-Jack-3" H 800 3950 50  0000 C CNN
-F 2 "" H 1150 3800 50  0001 C CNN
-F 3 "~" H 1150 3800 50  0001 C CNN
-	1    900  3700
-	1    0    0    -1
-$EndComp
-$Comp
 L Connector_Specialized:Jack-DC J1
 U 1 1 5ACC4F8C
@@
 F 0 "J1" H 800 2450 50  0000 R CNN
 F 1 "Jack-DC" H 950 2850 50  0000 R CNN
-F 2 "" H 850 2610 50  0001 C CNN
+F 2 "Connector_Audio:Jack_Horizontal" H 850 2610 50  0001 C CNN
 F 3 "~" H 850 2610 50  0001 C CNN
 	1    800  2650
@@
 	1    0    0    -1
 $EndComp
-Wire Wire Line
-	10400 3000 10400 3200
 Wire Wire Line
 	6000 3000 5900 3000
@@
 F 0 "Q1" H 3441 3846 50  0000 L CNN
 F 1 "2N2222" H 3441 3755 50  0000 L CNN
-F 2 "Package_TO_SOT_THT:TO-18" H 3450 3725 50  0001 L CIN
+F 2 "Package_TO_SOT_THT:TO-18-3" H 3450 3725 50  0001 L CIN
 F 3 "https://www.centralsemi.com/get_document.php?cmp=1&mergetype=pd&mergepath=pd&pdf_id=2N2221.PDF" H 3250 3800 50  0001 L CNN
 	1    3250 3800
@@
 F 0 "U1" H 9950 2533 50  0000 C CNN
 F 1 "foot_switch" H 9950 2624 50  0000 C CNN
-F 2 "" H 9950 3000 50  0001 C CNN
+F 2 "clasicOverdrive:FS57003PLT2B2M2QE" H 9950 3000 50  0001 C CNN
 F 3 "" H 9950 3000 50  0001 C CNN
 	3    9950 3000
@@
 F 0 "U1" H 1650 3942 50  0000 C CNN
 F 1 "foot_switch" H 1650 3851 50  0000 C CNN
-F 2 "" H 1650 3700 50  0001 C CNN
+F 2 "clasicOverdrive:FS57003PLT2B2M2QE" H 1650 3700 50  0001 C CNN
 F 3 "" H 1650 3700 50  0001 C CNN
 	2    1650 3700
@@
 L power:GND #PWR0126
 U 1 1 5ADBE742
-P 700 3900
-F 0 "#PWR0126" H 700 3650 50  0001 C CNN
-F 1 "GND" H 705 3727 50  0000 C CNN
-F 2 "" H 700 3900 50  0001 C CNN
-F 3 "" H 700 3900 50  0001 C CNN
-	1    700  3900
-	1    0    0    -1
-$EndComp
-Wire Wire Line
-	700  3900 700  3800
+P 1200 3900
+F 0 "#PWR0126" H 1200 3650 50  0001 C CNN
+F 1 "GND" H 1205 3727 50  0000 C CNN
+F 2 "" H 1200 3900 50  0001 C CNN
+F 3 "" H 1200 3900 50  0001 C CNN
+	1    1200 3900
+	1    0    0    -1
+$EndComp
+Wire Wire Line
+	1200 3900 1200 3800
 $Comp
 L clasicOverdrive:foot_switch U1
@@
 F 0 "U1" H 950 5583 50  0000 C CNN
 F 1 "foot_switch" H 950 5674 50  0000 C CNN
-F 2 "" H 950 6050 50  0001 C CNN
+F 2 "clasicOverdrive:FS57003PLT2B2M2QE" H 950 6050 50  0001 C CNN
 F 3 "" H 950 6050 50  0001 C CNN
 	1    950  6050
@@
 Wire Wire Line
 	650  6200 650  5950
-Wire Wire Line
-	1100 2750 1100 3600
 $Comp
 L power:+9V #PWR0128
@@
 Wire Wire Line
 	9650 1150 9650 2800
-Connection ~ 1350 3700
 Wire Wire Line
 	1350 1150 1350 3700
 Wire Wire Line
 	1350 1150 9650 1150
-Wire Wire Line
-	1100 3700 1350 3700
 Wire Wire Line
 	1250 5850 1350 5850
@@
 Text Notes 4500 2300 0    50   ~ 0
 DRIVE
+Text Notes 7300 2550 0    50   ~ 0
+LEVEL
+$Comp
+L dk_Barrel-Audio-Connectors:SN49B12B CON1
+U 1 1 5AD02C8E
+P 800 3700
+F 0 "CON1" H 856 4087 60  0000 C CNN
+F 1 "SN49B12B" H 856 3981 60  0000 C CNN
+F 2 "digikey-footprints:Headphone_Jack_6.35mm_RA49B14B" H 1000 3900 60  0001 L CNN
+F 3 "http://www.switchcraft.com/Drawings/SN49B_SERIES_CD.pdf" H 1000 4000 60  0001 L CNN
+F 4 "SC1522-ND" H 1000 4100 60  0001 L CNN "Digi-Key_PN"
+F 5 "SN49B12B" H 1000 4200 60  0001 L CNN "MPN"
+F 6 "Connectors, Interconnects" H 1000 4300 60  0001 L CNN "Category"
+F 7 "Barrel - Audio Connectors" H 1000 4400 60  0001 L CNN "Family"
+F 8 "http://www.switchcraft.com/Drawings/SN49B_SERIES_CD.pdf" H 1000 4500 60  0001 L CNN "DK_Datasheet_Link"
+F 9 "/product-detail/en/switchcraft-inc/SN49B12B/SC1522-ND/412780" H 1000 4600 60  0001 L CNN "DK_Detail_Page"
+F 10 "CONN JACK STEREO 6.35MM R/A" H 1000 4700 60  0001 L CNN "Description"
+F 11 "Switchcraft Inc." H 1000 4800 60  0001 L CNN "Manufacturer"
+F 12 "Active" H 1000 4900 60  0001 L CNN "Status"
+	1    800  3700
+	1    0    0    -1
+$EndComp
+$Comp
+L dk_Barrel-Audio-Connectors:SN49B12B CON2
+U 1 1 5AD030A4
+P 10800 3000
+F 0 "CON2" H 10857 3387 60  0000 C CNN
+F 1 "SN49B12B" H 10857 3281 60  0000 C CNN
+F 2 "digikey-footprints:Headphone_Jack_6.35mm_RA49B14B" H 11000 3200 60  0001 L CNN
+F 3 "http://www.switchcraft.com/Drawings/SN49B_SERIES_CD.pdf" H 11000 3300 60  0001 L CNN
+F 4 "SC1522-ND" H 11000 3400 60  0001 L CNN "Digi-Key_PN"
+F 5 "SN49B12B" H 11000 3500 60  0001 L CNN "MPN"
+F 6 "Connectors, Interconnects" H 11000 3600 60  0001 L CNN "Category"
+F 7 "Barrel - Audio Connectors" H 11000 3700 60  0001 L CNN "Family"
+F 8 "http://www.switchcraft.com/Drawings/SN49B_SERIES_CD.pdf" H 11000 3800 60  0001 L CNN "DK_Datasheet_Link"
+F 9 "/product-detail/en/switchcraft-inc/SN49B12B/SC1522-ND/412780" H 11000 3900 60  0001 L CNN "DK_Detail_Page"
+F 10 "CONN JACK STEREO 6.35MM R/A" H 11000 4000 60  0001 L CNN "Description"
+F 11 "Switchcraft Inc." H 11000 4100 60  0001 L CNN "Manufacturer"
+F 12 "Active" H 11000 4200 60  0001 L CNN "Status"
+	1    10800 3000
+	-1   0    0    -1
+$EndComp
+Wire Wire Line
+	1100 2750 1200 2750
+Wire Wire Line
+	1200 2750 1200 3600
+Wire Wire Line
+	1200 3700 1350 3700
+Connection ~ 1350 3700
+Wire Wire Line
+	10400 3100 10400 3200
 $EndSCHEMATC

Commit message: Board Finished
Parts:
- added MK1, MK2, MK3, MK4: Mounting_Hole, MountingHole:MountingHole_3.2mm_M3, symbol Mechanical:Mounting_Hole
Changed lines of the file:
@@
 Wire Wire Line
 	10400 3100 10400 3200
+$Comp
+L Mechanical:Mounting_Hole MK1
+U 1 1 5ADA8A7E
+P 9700 5150
+F 0 "MK1" H 9800 5196 50  0000 L CNN
+F 1 "Mounting_Hole" H 9800 5105 50  0000 L CNN
+F 2 "MountingHole:MountingHole_3.2mm_M3" H 9700 5150 50  0001 C CNN
+F 3 "" H 9700 5150 50  0001 C CNN
+	1    9700 5150
+	1    0    0    -1
+$EndComp
+$Comp
+L Mechanical:Mounting_Hole MK2
+U 1 1 5ADA8C59
+P 9700 5350
+F 0 "MK2" H 9800 5396 50  0000 L CNN
+F 1 "Mounting_Hole" H 9800 5305 50  0000 L CNN
+F 2 "MountingHole:MountingHole_3.2mm_M3" H 9700 5350 50  0001 C CNN
+F 3 "" H 9700 5350 50  0001 C CNN
+	1    9700 5350
+	1    0    0    -1
+$EndComp
+$Comp
+L Mechanical:Mounting_Hole MK3
+U 1 1 5ADA8CDF
+P 9700 5550
+F 0 "MK3" H 9800 5596 50  0000 L CNN
+F 1 "Mounting_Hole" H 9800 5505 50  0000 L CNN
+F 2 "MountingHole:MountingHole_3.2mm_M3" H 9700 5550 50  0001 C CNN
+F 3 "" H 9700 5550 50  0001 C CNN
+	1    9700 5550
+	1    0    0    -1
+$EndComp
+$Comp
+L Mechanical:Mounting_Hole MK4
+U 1 1 5ADA8D59
+P 9700 5750
+F 0 "MK4" H 9800 5796 50  0000 L CNN
+F 1 "Mounting_Hole" H 9800 5705 50  0000 L CNN
+F 2 "MountingHole:MountingHole_3.2mm_M3" H 9700 5750 50  0001 C CNN
+F 3 "" H 9700 5750 50  0001 C CNN
+	1    9700 5750
+	1    0    0    -1
+$EndComp
 $EndSCHEMATC

Commit message: updated bom and footprint for the diodes@
Parts:
- CON1, CON2: symbol dk_Barrel-Audio-Connectors:SN49B12B -> clasicOverdrive-rescue:SN49B12B-dk_Barrel-Audio-Connectors
- J1: symbol Connector_Specialized:Jack-DC -> clasicOverdrive-rescue:Jack-DC-Connector_Specialized
- RV1, RV2, RV3: symbol Device:POT -> clasicOverdrive-rescue:POT-Device
Changed lines of the file:
@@
 $EndComp
 $Comp
-L Device:POT RV3
+L clasicOverdrive-rescue:POT-Device RV3
 U 1 1 5ACC9FDB
 P 7550 2750
@@
 $EndComp
 $Comp
-L Device:POT RV2
+L clasicOverdrive-rescue:POT-Device RV2
 U 1 1 5ACC2718
 P 5550 1600
@@
 $EndComp
 $Comp
-L Device:POT RV1
+L clasicOverdrive-rescue:POT-Device RV1
 U 1 1 5ACC2B71
 P 4550 2550
@@
 $EndComp
 $Comp
-L Connector_Specialized:Jack-DC J1
+L clasicOverdrive-rescue:Jack-DC-Connector_Specialized J1
 U 1 1 5ACC4F8C
 P 800 2650
@@
 LEVEL
 $Comp
-L dk_Barrel-Audio-Connectors:SN49B12B CON1
+L clasicOverdrive-rescue:SN49B12B-dk_Barrel-Audio-Connectors CON1
 U 1 1 5AD02C8E
 P 800 3700
@@
 $EndComp
 $Comp
-L dk_Barrel-Audio-Connectors:SN49B12B CON2
+L clasicOverdrive-rescue:SN49B12B-dk_Barrel-Audio-Connectors CON2
 U 1 1 5AD030A4
 P 10800 3000

Commit message: bom
Parts:
- D2, D3: footprint Diode_SMD:D_0805_2012Metric_Pad0.97x1.50mm_HandSolder -> Diode_SMD:D_SOD-323_HandSoldering
Changed lines of the file:
@@
 F 0 "D2" H 4350 1816 50  0000 C CNN
 F 1 "1N4148" H 4350 1725 50  0000 C CNN
-F 2 "Diode_SMD:D_0805_2012Metric_Pad0.97x1.50mm_HandSolder" H 4350 1425 50  0001 C CNN
+F 2 "Diode_SMD:D_SOD-323_HandSoldering" H 4350 1425 50  0001 C CNN
 F 3 "http://www.nxp.com/documents/data_sheet/1N4148_1N4448.pdf" H 4350 1600 50  0001 C CNN
 	1    4350 1600
@@
 F 0 "D3" H 4350 1784 50  0000 C CNN
 F 1 "1N4148" H 4350 1875 50  0000 C CNN
-F 2 "Diode_SMD:D_0805_2012Metric_Pad0.97x1.50mm_HandSolder" H 4350 1825 50  0001 C CNN
+F 2 "Diode_SMD:D_SOD-323_HandSoldering" H 4350 1825 50  0001 C CNN
 F 3 "http://www.nxp.com/documents/data_sheet/1N4148_1N4448.pdf" H 4350 2000 50  0001 C CNN
 	1    4350 2000

Commit message: update pcb and schematic with pads
Parts:
- added TP1: 9V, TestPoint:TestPoint_Pad_D2.0mm, symbol Connector:TestPoint
- added TP2: 4V5, TestPoint:TestPoint_Pad_D2.0mm, symbol Connector:TestPoint
- added unit 3 of U2
- MK1, MK2, MK3, MK4: symbol Mechanical:Mounting_Hole -> clasicOverdrive-rescue:Mounting_Hole-Mechanical
Connections:
- wire segments 119 -> 115
Changed lines of the file:
@@
 EESchema Schematic File Version 4
 LIBS:clasicOverdrive-cache
-EELAYER 26 0
+EELAYER 29 0
 EELAYER END
 $Descr A4 11693 8268
@@
 	1600 5200 1600 5050
 $Comp
-L power:+9V #PWR0122
-U 1 1 5AD25683
-P 6200 3500
-F 0 "#PWR0122" H 6200 3350 50  0001 C CNN
-F 1 "+9V" H 6215 3673 50  0000 C CNN
-F 2 "" H 6200 3500 50  0001 C CNN
-F 3 "" H 6200 3500 50  0001 C CNN
-	1    6200 3500
-	-1   0    0    1
-$EndComp
-Wire Wire Line
-	6200 3500 6200 3400
-$Comp
-L power:GND #PWR0123
-U 1 1 5AD28C8D
-P 6200 2650
-F 0 "#PWR0123" H 6200 2400 50  0001 C CNN
-F 1 "GND" H 6205 2477 50  0000 C CNN
-F 2 "" H 6200 2650 50  0001 C CNN
-F 3 "" H 6200 2650 50  0001 C CNN
-	1    6200 2650
-	-1   0    0    1
-$EndComp
-Wire Wire Line
-	6200 2650 6200 2800
-$Comp
 L power:GND #PWR0124
 U 1 1 5AD2C63D
-P 4250 3550
-F 0 "#PWR0124" H 4250 3300 50  0001 C CNN
-F 1 "GND" H 4255 3377 50  0000 C CNN
-F 2 "" H 4250 3550 50  0001 C CNN
-F 3 "" H 4250 3550 50  0001 C CNN
-	1    4250 3550
-	-1   0    0    1
-$EndComp
-Wire Wire Line
-	4250 3550 4250 3650
+P 3900 6450
+F 0 "#PWR0124" H 3900 6200 50  0001 C CNN
+F 1 "GND" H 3905 6277 50  0000 C CNN
+F 2 "" H 3900 6450 50  0001 C CNN
+F 3 "" H 3900 6450 50  0001 C CNN
+	1    3900 6450
+	1    0    0    -1
+$EndComp
 $Comp
 L Device:C C4
@@
 L power:+9V #PWR0125
 U 1 1 5AD5279F
-P 4250 4350
-F 0 "#PWR0125" H 4250 4200 50  0001 C CNN
-F 1 "+9V" H 4265 4523 50  0000 C CNN
-F 2 "" H 4250 4350 50  0001 C CNN
-F 3 "" H 4250 4350 50  0001 C CNN
-	1    4250 4350
-	-1   0    0    1
-$EndComp
-Wire Wire Line
-	4250 4350 4250 4250
+P 3900 5850
+F 0 "#PWR0125" H 3900 5700 50  0001 C CNN
+F 1 "+9V" H 3915 6023 50  0000 C CNN
+F 2 "" H 3900 5850 50  0001 C CNN
+F 3 "" H 3900 5850 50  0001 C CNN
+	1    3900 5850
+	1    0    0    -1
+$EndComp
 Wire Wire Line
 	4800 3200 4500 3200
@@
 	10400 3100 10400 3200
 $Comp
-L Mechanical:Mounting_Hole MK1
+L clasicOverdrive-rescue:Mounting_Hole-Mechanical MK1
 U 1 1 5ADA8A7E
 P 9700 5150
@@
 $EndComp
 $Comp
-L Mechanical:Mounting_Hole MK2
+L clasicOverdrive-rescue:Mounting_Hole-Mechanical MK2
 U 1 1 5ADA8C59
 P 9700 5350
@@
 $EndComp
 $Comp
-L Mechanical:Mounting_Hole MK3
+L clasicOverdrive-rescue:Mounting_Hole-Mechanical MK3
 U 1 1 5ADA8CDF
 P 9700 5550
@@
 $EndComp
 $Comp
-L Mechanical:Mounting_Hole MK4
+L clasicOverdrive-rescue:Mounting_Hole-Mechanical MK4
 U 1 1 5ADA8D59
 P 9700 5750
@@
 	1    0    0    -1
 $EndComp
+$Comp
+L Amplifier_Operational:LM4562 U2
+U 3 1 5BE39832
+P 4000 6150
+F 0 "U2" H 3958 6196 50  0000 L CNN
+F 1 "LM4562" H 3958 6105 50  0000 L CNN
+F 2 "Package_SO:SOIC-8_3.9x4.9mm_P1.27mm" H 4000 6150 50  0001 C CNN
+F 3 "http://www.ti.com/lit/ds/symlink/lm4562.pdf" H 4000 6150 50  0001 C CNN
+	3    4000 6150
+	1    0    0    -1
+$EndComp
+$Comp
+L Connector:TestPoint TP1
+U 1 1 5BE3E2A4
+P 7350 5650
+F 0 "TP1" H 7292 5676 50  0000 R CNN
+F 1 "9V" H 7292 5767 50  0000 R CNN
+F 2 "TestPoint:TestPoint_Pad_D2.0mm" H 7550 5650 50  0001 C CNN
+F 3 "~" H 7550 5650 50  0001 C CNN
+	1    7350 5650
+	-1   0    0    1
+$EndComp
+$Comp
+L power:+9V #PWR0122
+U 1 1 5BE3EBEA
+P 7350 5650
+F 0 "#PWR0122" H 7350 5500 50  0001 C CNN
+F 1 "+9V" H 7365 5823 50  0000 C CNN
+F 2 "" H 7350 5650 50  0001 C CNN
+F 3 "" H 7350 5650 50  0001 C CNN
+	1    7350 5650
+	1    0    0    -1
+$EndComp
+$Comp
+L Connector:TestPoint TP2
+U 1 1 5BE3F090
+P 7850 5650
+F 0 "TP2" H 7792 5676 50  0000 R CNN
+F 1 "4V5" H 7792 5767 50  0000 R CNN
+F 2 "TestPoint:TestPoint_Pad_D2.0mm" H 8050 5650 50  0001 C CNN
+F 3 "~" H 8050 5650 50  0001 C CNN
+	1    7850 5650
+	-1   0    0    1
+$EndComp
+$Comp
+L clasicOverdrive:+4V5 #PWR0123
+U 1 1 5BE3F2E8
+P 7850 5650
+F 0 "#PWR0123" H 7850 5500 50  0001 C CNN
+F 1 "+4V5" H 7865 5823 50  0000 C CNN
+F 2 "" H 7850 5650 50  0001 C CNN
+F 3 "" H 7850 5650 50  0001 C CNN
+	1    7850 5650
+	1    0    0    -1
+$EndComp

Commit message: Rev A
Parts:
- removed CON1, CON2: SN49B12B, digikey-footprints:Headphone_Jack_6.35mm_RA49B14B, symbol clasicOverdrive-rescue:SN49B12B-dk_Barrel-Audio-Connectors
- removed MK1, MK2, MK3, MK4: Mounting_Hole, MountingHole:MountingHole_3.2mm_M3, symbol clasicOverdrive-rescue:Mounting_Hole-Mechanical
- added C12: 1u, Capacitor_SMD:C_0805_2012Metric, symbol Device:C
- added C13, C14, C15, C16: 0.1u, Capacitor_SMD:C_0805_2012Metric, symbol Device:C
- added FID1, FID2, FID3: Fiducial, Fiducial:Fiducial_1mm_Mask2mm, symbol Mechanical:Fiducial
- added H1, H2, H3, H4: MountingHole_Pad, MountingHole:MountingHole_2.7mm_M2.5_Pad_Via, symbol Mechanical:MountingHole_Pad
- added J2, J3: AudioJack3_Switch, clasicOverdrive:Jack_6.35mm_Amphenol_ACJS-MHOM, symbol Connector:AudioJack3_Switch
- added T1: LA_LOGO, clasicOverdrive:LA_LOGO_MASK, symbol clasicOverdrive:LA_LOGO
- C1: footprint Capacitor_SMD:C_0805_2012Metric_Pad1.15x1.50mm_HandSolder -> Capacitor_SMD:C_0805_2012Metric; Digi-Key (none) -> 399-1163-1-ND; manf# (none) -> C0805C223K5RACTU
- C10: footprint Capacitor_SMD:C_0805_2012Metric_Pad1.15x1.50mm_HandSolder -> Capacitor_SMD:C_0805_2012Metric; Digi-Key (none) -> 399-8000-1-ND; manf# (none) -> C0805C104M3RACTU
- C11: footprint Capacitor_SMD:C_1206_3216Metric_Pad1.24x1.80mm_HandSolder -> Capacitor_SMD:C_1206_3216Metric; Digi-Key (none) -> 478-10743-1-ND; manf# (none) -> TAJA106K016RNJV
- C2: footprint Capacitor_SMD:C_0805_2012Metric_Pad1.15x1.50mm_HandSolder -> Capacitor_SMD:C_0805_2012Metric; Digi-Key (none) -> 1276-2527-1-ND; manf# (none) -> CL21B473KBANNNC
- C3, C9: footprint Capacitor_SMD:C_0805_2012Metric_Pad1.15x1.50mm_HandSolder -> Capacitor_SMD:C_0805_2012Metric; Digi-Key (none) -> 1276-6471-1-ND; manf# (none) -> CL21B105KOFNNNG
- C4: footprint Capacitor_SMD:C_0805_2012Metric_Pad1.15x1.50mm_HandSolder -> Capacitor_SMD:C_0805_2012Metric; Digi-Key (none) -> 1276-2670-1-ND; manf# (none) -> CL21C510JBANNNC
- C5: footprint Capacitor_SMD:C_1206_3216Metric_Pad1.24x1.80mm_HandSolder -> Capacitor_Tantalum_SMD:CP_EIA-6032-28_Kemet-C; Digi-Key (none) -> 399-11392-1-ND; manf# (none) -> T495C107K016ATE200
- C6, C7: footprint Capacitor_SMD:C_1206_3216Metric_Pad1.24x1.80mm_HandSolder -> Capacitor_Tantalum_SMD:CP_EIA-2012-12_Kemet-R; Digi-Key (none) -> 718-2502-1-ND; manf# (none) -> TMCP1D224MTRF
- C8: footprint Capacitor_SMD:C_1206_3216Metric_Pad1.24x1.80mm_HandSolder -> Capacitor_Tantalum_SMD:CP_EIA-3216-18_Kemet-A; Digi-Key (none) -> 718-2387-1-ND; manf# (none) -> TMCMA1A476MTRF
- D1: footprint LED_SMD:LED_1206_3216Metric_Pad1.07x1.80mm_HandSolder -> LED_SMD:LED_1206_3216Metric; Digi-Key (none) -> 732-4989-1-ND; manf# (none) -> 150120BS75000
- D2, D3: Digi-Key (none) -> 1N4148WXTPMSCT-ND; manf# (none) -> 1N4148WX-TP
- J1: footprint Connector_Audio:Jack_Horizontal -> Connector_BarrelJack:BarrelJack_Horizontal; symbol clasicOverdrive-rescue:Jack-DC-Connector_Specialized -> Connector:Barrel_Jack_Switch; Digi-Key (none) -> CP-002A-ND; manf# (none) -> PJ-002A
- Q1, Q2: Digi-Key (none) -> 1514-2N2222APBFREE-ND; manf# (none) -> 2N2222A PBFREE
- R1, R6: footprint Resistor_SMD:R_0603_1608Metric_Pad0.84x1.00mm_HandSolder -> Resistor_SMD:R_0603_1608Metric; Digi-Key (none) -> 311-4.70KHRCT-ND; manf# (none) -> RC0603FR-074K7L
- R10, R11, R13, R17, R19, R5, R7: footprint Resistor_SMD:R_0603_1608Metric_Pad0.84x1.00mm_HandSolder -> Resistor_SMD:R_0603_1608Metric; Digi-Key (none) -> 311-10.0KHRCT-ND; manf# (none) -> RC0603FR-0710KL
- R12: footprint Resistor_SMD:R_0603_1608Metric_Pad0.84x1.00mm_HandSolder -> Resistor_SMD:R_0603_1608Metric; Digi-Key (none) -> 311-220HRCT-ND; manf# (none) -> RC0603FR-07220RL
- R14, R15, R3, R9: footprint Resistor_SMD:R_0603_1608Metric_Pad0.84x1.00mm_HandSolder -> Resistor_SMD:R_0603_1608Metric; Digi-Key (none) -> 311-1.00KHRCT-ND; manf# (none) -> RC0603FR-071KL
- R16, R2, R4: footprint Resistor_SMD:R_0603_1608Metric_Pad0.84x1.00mm_HandSolder -> Resistor_SMD:R_0603_1608Metric; Digi-Key (none) -> 311-511KHRCT-ND; manf# (none) -> RC0603FR-07511KL
- R18: footprint Resistor_SMD:R_0603_1608Metric_Pad0.84x1.00mm_HandSolder -> Resistor_SMD:R_0603_1608Metric; Digi-Key (none) -> 311-100HRCT-ND; manf# (none) -> RC0603FR-07100RL
- R8: footprint Resistor_SMD:R_0603_1608Metric_Pad0.84x1.00mm_HandSolder -> Resistor_SMD:R_0603_1608Metric; Digi-Key (none) -> YAG3616CT-ND; manf# (none) -> AC0603FR-0751KL
- RV1: footprint clasicOverdrive:Pot_series_296 -> Potentiometer_THT:Potentiometer_Bourns_PTV09A-1_Single_Vertical; symbol clasicOverdrive-rescue:POT-Device -> Device:R_POT; Digi-Key (none) -> PTV09A-4020F-A504-ND; Info (none) -> DRIVE; manf# (none) -> PTV09A-4020F-A504
- RV2: footprint clasicOverdrive:Pot_series_296 -> Potentiometer_THT:Potentiometer_Bourns_PTV09A-1_Single_Vertical; symbol clasicOverdrive-rescue:POT-Device -> Device:R_POT; Digi-Key (none) -> PTV09A-4020F-B203-ND; Info (none) -> TONE; manf# (none) -> PTV09A-4020F-B203
- RV3: footprint clasicOverdrive:Pot_series_296 -> Potentiometer_THT:Potentiometer_Bourns_PTV09A-1_Single_Vertical; symbol clasicOverdrive-rescue:POT-Device -> Device:R_POT; Digi-Key (none) -> PTV09A-4020F-B104-ND; Info (none) -> LEVEL; manf# (none) -> PTV09A-4020F-B104
- TP1, TP2: footprint TestPoint:TestPoint_Pad_D2.0mm -> TestPoint:TestPoint_Pad_D1.5mm
- U1: footprint clasicOverdrive:FS57003PLT2B2M2QE -> clasicOverdrive:Foot_Switch_E-Switch_FS57003PLT2B2M2QE; Digi-Key (none) -> EG5492-ND; manf# (none) -> FS57003PLT2B2M2QE
- U2: Digi-Key (none) -> 296-35279-1-ND; manf# (none) -> LM4562MAX/NOPB
Connections:
- net +4V5: now also C14.1, C15.1, C16.1
- net +9V: now also C12.1, C13.1
- net GND: now also C12.2, C13.2, C14.2, C15.2, C16.2, H1.1, H2.1, H3.1, H4.1, J2.S, J3.S
- net at R14.2, U2.6 (-): now also RV2.3; no longer RV2.1
- net at C6.1, R13.1, R9.1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: now also RV2.1; no longer RV2.3
- net at RV1.1: now also C4.2, D2.2 (A), D3.1 (K), R9.2, RV1.2, U2.1; no longer R8.1
- net GNDPWR: now reaches J1.1
- net GNDPWR: now also J2.R
- net at U1.4, U1.9: now also J2.T
- net at U1.8: now also J3.R
- new net: R8.1, RV1.3
- no-connect marks 0 -> 8
Other:
- note removed: "DRIVE"
- note removed: "LEVEL"
- note removed: "TONE"
- moved on the sheet: C5, C8, R10, R11, TP1, U2C
